File: peakdetector/peakdetector.sch (KiCad schematic (older format))
At the start: 11 parts, among them J1 Conn_01x07_Male, U1 TL074

Commit message: Switch to LM324.
Parts:
- U1: value TL074 -> LM324
Changed lines of the file:
@@
 P 2600 3050
 F 0 "J1" H 2706 3528 50  0000 C CNN
-F 1 "Conn_01x07_Male" H 2706 3437 50  0000 C CNN
+F 1 "Conn_01x07_Male" H 2706 3437 50  0001 C CNN
 F 2 "Pin_Headers:Pin_Header_Straight_1x07_Pitch2.54mm" H 2600 3050 50  0001 C CNN
 F 3 "~" H 2600 3050 50  0001 C CNN
@@
 P 3500 2350
 F 0 "U1" H 3450 2350 50  0000 C CNN
-F 1 "TL074" H 3500 2626 50  0000 C CNN
+F 1 "LM324" H 3500 2626 50  0000 C CNN
 F 2 "peakdetector:SOP14" H 3450 2450 50  0001 C CNN
 F 3 "http://www.ti.com/lit/ds/symlink/tl071.pdf" H 3550 2550 50  0001 C CNN
@@
 P 5200 2250
 F 0 "U1" H 5150 2250 50  0000 C CNN
-F 1 "TL074" H 5200 2526 50  0000 C CNN
+F 1 "LM324" H 5200 2526 50  0000 C CNN
 F 2 "peakdetector:SOP14" H 5150 2350 50  0001 C CNN
 F 3 "http://www.ti.com/lit/ds/symlink/tl071.pdf" H 5250 2450 50  0001 C CNN
@@
 P 3500 4000
 F 0 "U1" H 3450 4000 50  0000 C CNN
-F 1 "TL074" H 3500 4276 50  0000 C CNN
+F 1 "LM324" H 3500 4276 50  0000 C CNN
 F 2 "peakdetector:SOP14" H 3450 4100 50  0001 C CNN
 F 3 "http://www.ti.com/lit/ds/symlink/tl071.pdf" H 3550 4200 50  0001 C CNN
@@
 P 5300 3900
 F 0 "U1" H 5250 3900 50  0000 C CNN
-F 1 "TL074" H 5300 4176 50  0000 C CNN
+F 1 "LM324" H 5300 4176 50  0000 C CNN
 F 2 "peakdetector:SOP14" H 5250 4000 50  0001 C CNN
 F 3 "http://www.ti.com/lit/ds/symlink/tl071.pdf" H 5350 4100 50  0001 C CNN
@@
 P 2950 5750
 F 0 "U1" H 2908 5796 50  0000 L CNN
-F 1 "TL074" H 2908 5705 50  0000 L CNN
+F 1 "LM324" H 2908 5705 50  0000 L CNN
 F 2 "peakdetector:SOP14" H 2900 5850 50  0001 C CNN
 F 3 "http://www.ti.com/lit/ds/symlink/tl071.pdf" H 3000 5950 50  0001 C CNN
