File: pcb/chairbot/chairbot.sch (KiCad schematic (older format))
At the start: 15 parts

Commit message: Work on schematic.
Parts:
- removed C? (x3): C, symbol Device:C
- removed D?: D_Schottky, symbol Device:D_Schottky
- removed J?: Conn_01x02, symbol Connector_Generic:Conn_01x02
- removed Q?: FDD8447, Package_TO_SOT_THT:TO-92_Inline, symbol Transistor_FET:BS107
- removed R?: R, symbol Device:R
- removed U? (x2): Motor_driver, symbol chairbot:Motor_driver
- removed U? (x2): 74HCT08, symbol 74xx_IEEE:7408
- added C?: C, symbol Device:C
- added C?: 10u, symbol Device:CP
- added D?: SS34, symbol Device:D_Schottky
- added F?: Fuse, symbol Device:Fuse
- added J?: Conn_01x02, symbol Connector_Generic:Conn_01x02
- added U?: 74HCT244, symbol 74xx:74HCT244
- added U?: buck-converter, mylib:buck-converter, symbol buckconverter:buck-converter
Connections:
- net labels added: +3.3V, PWM_A_L, PWM_A_R, PWM_B_L, PWM_B_R
- wire segments 41 -> 36
Other:
- note added: "24V IN"
- note removed: "Brake"

Commit message: Add nRF24L01.
Parts:
- added U?: nRF24L01+, MODULE, symbol nRF24L01:nRF24L01+
Changed lines of the file:
@@
 	7850 6050 7850 5950
 Connection ~ 7850 5950
+$Comp
+L nRF24L01:nRF24L01+ U?
+U 1 1 5BD22025
+P 5850 3850
+F 0 "U?" H 5850 4365 50  0000 C CNN
+F 1 "nRF24L01+" H 5850 4274 50  0000 C CNN
+F 2 "MODULE" H 5850 3950 50  0001 C CNN
+F 3 "DOCUMENTATION" H 5850 3800 50  0001 C CNN
+	1    5850 3850
+	1    0    0    -1
+$EndComp
 $EndSCHEMATC

Commit message: Work.
Parts:
- added C2: 100n, Capacitor_SMD:C_0603_1608Metric, symbol Device:C
- added C3: 10u, Capacitor_SMD:C_0805_2012Metric, symbol Device:C
- C1: renamed from C?; value C -> 100n; footprint (none) -> Capacitor_SMD:C_0603_1608Metric
- C4: renamed from C?; footprint (none) -> Capacitor_SMD:C_0805_2012Metric
- D1: renamed from D?; footprint (none) -> Diode_SMD:D_SMC
- F1: renamed from F?; footprint (none) -> Resistor_THT:R_Axial_DIN0309_L9.0mm_D3.2mm_P2.54mm_Vertical
- J1: renamed from J?; footprint (none) -> Connector_JST:JST_XH_B02B-XH-A_1x02_P2.50mm_Vertical
- J2: renamed from J?; footprint (none) -> Connector_JST:JST_XH_B05B-XH-A_1x05_P2.50mm_Vertical
- U1: renamed from U?; footprint ESP32mini:ESP32mini -> chairbot:ESP32mini
- U2: renamed from U?; footprint (none) -> Package_SO:TSSOP-14_4.4x5mm_P0.65mm
- U3: renamed from U?; footprint (none) -> Package_SO:TSSOP-20_4.4x6.5mm_P0.65mm
- U4: renamed from U?; footprint mylib:buck-converter -> chairbot:buck-converter
- U5: renamed from U?; footprint MODULE -> chairbot:nRF24L01
Connections:
- net labels added: +3V3, +5C, Brake, CE, CS, ENA, ENB, MISO, MOSI, SCK, SCL, SDA
- wire segments 36 -> 60
- no-connect marks 0 -> 1

Commit message: Work work work.
Parts:
- added C8: 100n, Capacitor_SMD:C_0603_1608Metric, symbol Device:C
- added unit 4 of U2
- added U8: AMS1117-3.3, Package_TO_SOT_SMD:SOT-223-3_TabPin2, symbol Regulator_Linear:AMS1117-3.3
- U2: footprint Package_SO:TSSOP-14_4.4x5mm_P0.65mm -> (none)
Connections:
- net labels added: EN
- net labels removed: +3V3, +5C, ENA, ENB
- wire segments 60 -> 74
- no-connect marks 1 -> 16
Changed lines of the file:
@@
 $Comp
 L 74xx_IEEE:7408 U2
-U 3 1 5BC3AC55
+U 2 1 5BC3AC55
 P 3350 5450
 F 0 "U2" H 3350 5815 50  0000 C CNN
 F 1 "74HCT08" H 3350 5724 50  0000 C CNN
-F 2 "Package_SO:TSSOP-14_4.4x5mm_P0.65mm" H 3350 5450 50  0001 C CNN
+F 2 "" H 3350 5450 50  0001 C CNN
 F 3 "" H 3350 5450 50  0001 C CNN
-	3    3350 5450
+	2    3350 5450
 	1    0    0    -1
 $EndComp
 $Comp
 L 74xx_IEEE:7408 U2
-U 4 1 5BC3ACB2
+U 3 1 5BC3ACB2
 P 3350 6250
 F 0 "U2" H 3350 6615 50  0000 C CNN
 F 1 "74HCT08" H 3350 6524 50  0000 C CNN
-F 2 "Package_SO:TSSOP-14_4.4x5mm_P0.65mm" H 3350 6250 50  0001 C CNN
+F 2 "" H 3350 6250 50  0001 C CNN
 F 3 "" H 3350 6250 50  0001 C CNN
-	4    3350 6250
+	3    3350 6250
 	1    0    0    -1
 $EndComp
@@
 	9900 3600 9750 3600
 $Comp
-L power:+3V3 #PWR04
-U 1 1 5BD247A9
-P 7250 3650
-F 0 "#PWR04" H 7250 3500 50  0001 C CNN
-F 1 "+3V3" H 7265 3823 50  0000 C CNN
-F 2 "" H 7250 3650 50  0001 C CNN
-F 3 "" H 7250 3650 50  0001 C CNN
-	1    7250 3650
-	1    0    0    -1
-$EndComp
-$Comp
 L Device:C C2
 U 1 1 5BD28A43
@@
 Wire Wire Line
 	7850 3350 8250 3350
-Wire Wire Line
-	7250 3650 7250 3750
 Wire Wire Line
 	7250 3750 7550 3750
@@
 Wire Wire Line
 	5150 3850 5450 3850
-$Comp
-L power:+5C #PWR01
-U 1 1 5BD2EB2D
-P 5450 3650
-F 0 "#PWR01" H 5450 3500 50  0001 C CNN
-F 1 "+5C" H 5465 3823 50  0000 C CNN
-F 2 "" H 5450 3650 50  0001 C CNN
-F 3 "" H 5450 3650 50  0001 C CNN
-	1    5450 3650
-	1    0    0    -1
-$EndComp
 Wire Wire Line
 	5450 3650 5450 3750
@@
 CS
 Text GLabel 1150 2150 0    50   Input ~ 0
-ENA
-Text GLabel 1150 2350 0    50   Input ~ 0
-ENB
+EN
 Text GLabel 1150 2800 0    50   Input ~ 0
 Brake
+$Comp
+L Regulator_Linear:AMS1117-3.3 U8
+U 1 1 5BD301D2
+P 6950 3750
+F 0 "U8" H 6950 3992 50  0000 C CNN
+F 1 "AMS1117-3.3" H 6950 3901 50  0000 C CNN
+F 2 "Package_TO_SOT_SMD:SOT-223-3_TabPin2" H 6950 3950 50  0001 C CNN
+F 3 "http://www.advanced-monolithic.com/pdf/ds1117.pdf" H 7050 3500 50  0001 C CNN
+	1    6950 3750
+	1    0    0    -1
+$EndComp
+$Comp
+L power:+5V #PWR04
+U 1 1 5BD30336
+P 6550 3600
+F 0 "#PWR04" H 6550 3450 50  0001 C CNN
+F 1 "+5V" H 6565 3773 50  0000 C CNN
+F 2 "" H 6550 3600 50  0001 C CNN
+F 3 "" H 6550 3600 50  0001 C CNN
+	1    6550 3600
+	1    0    0    -1
+$EndComp
+Wire Wire Line
+	6550 3600 6550 3750
+Wire Wire Line
+	6550 3750 6650 3750
+$Comp
+L power:GND #PWR08
+U 1 1 5BD311D3
+P 6950 4150
+F 0 "#PWR08" H 6950 3900 50  0001 C CNN
+F 1 "GND" H 6955 3977 50  0000 C CNN
+F 2 "" H 6950 4150 50  0001 C CNN
+F 3 "" H 6950 4150 50  0001 C CNN
+	1    6950 4150
+	1    0    0    -1
+$EndComp
+Wire Wire Line
+	6950 4150 6950 4100
+$Comp
+L Device:C C8
+U 1 1 5BD320D0
+P 6550 3950
+F 0 "C8" H 6665 3996 50  0000 L CNN
+F 1 "100n" H 6665 3905 50  0000 L CNN
+F 2 "Capacitor_SMD:C_0603_1608Metric" H 6588 3800 50  0001 C CNN
+F 3 "~" H 6550 3950 50  0001 C CNN
+	1    6550 3950
+	1    0    0    -1
+$EndComp
+Wire Wire Line
+	6550 4100 6950 4100
+Connection ~ 6950 4100
+Wire Wire Line
+	6950 4100 6950 4050
+Wire Wire Line
+	6550 3750 6550 3800
+Connection ~ 6550 3750
+$Comp
+L 74xx_IEEE:7408 U2
+U 4 1 5BD46086
+P 3350 7150
+F 0 "U2" H 3350 7515 50  0000 C CNN
+F 1 "74HCT08" H 3350 7424 50  0000 C CNN
+F 2 "" H 3350 7150 50  0001 C CNN
+F 3 "" H 3350 7150 50  0001 C CNN
+	4    3350 7150
+	1    0    0    -1
+$EndComp
+NoConn ~ 3900 5450
+NoConn ~ 3900 6250
+NoConn ~ 3900 7150
+$Comp
+L power:+5V #PWR0117
+U 1 1 5BD4A3E6
+P 2400 6850
+F 0 "#PWR0117" H 2400 6700 50  0001 C CNN
+F 1 "+5V" H 2415 7023 50  0000 C CNN
+F 2 "" H 2400 6850 50  0001 C CNN
+F 3 "" H 2400 6850 50  0001 C CNN
+	1    2400 6850
+	1    0    0    -1
+$EndComp
+Wire Wire Line
+	2400 6850 2400 7050
+Wire Wire Line
+	2400 7250 2800 7250
+Wire Wire Line
+	2800 7050 2400 7050
+Connection ~ 2400 7050
+Wire Wire Line
+	2400 7050 2400 7250
+$Comp
+L power:GND #PWR0118
+U 1 1 5BD4C883
+P 2400 5750
+F 0 "#PWR0118" H 2400 5500 50  0001 C CNN
+F 1 "GND" H 2405 5577 50  0000 C CNN
+F 2 "" H 2400 5750 50  0001 C CNN
+F 3 "" H 2400 5750 50  0001 C CNN
+	1    2400 5750
+	1    0    0    -1
+$EndComp
+Wire Wire Line
+	2400 5750 2400 5550
+Wire Wire Line
+	2400 5350 2800 5350
+Wire Wire Line
+	2800 5550 2400 5550
+Connection ~ 2400 5550
+Wire Wire Line
+	2400 5550 2400 5350
+NoConn ~ 4150 1700
+NoConn ~ 4150 1800
+NoConn ~ 4150 1900
+NoConn ~ 4150 2000
+NoConn ~ 4150 2100
+NoConn ~ 4150 2200
+NoConn ~ 4150 2300
+NoConn ~ 4150 2400
+NoConn ~ 4150 2500
+NoConn ~ 2200 3100
+NoConn ~ 2200 3300
+NoConn ~ 2200 3400
+$Comp
+L power:PWR_FLAG #FLG0101
+U 1 1 5BD6032C
+P 9150 5450
+F 0 "#FLG0101" H 9150 5525 50  0001 C CNN
+F 1 "PWR_FLAG" H 9150 5624 50  0000 C CNN
+F 2 "" H 9150 5450 50  0001 C CNN
+F 3 "~" H 9150 5450 50  0001 C CNN
+	1    9150 5450
+	1    0    0    -1
+$EndComp
+$Comp
+L power:+24V #PWR0119
+U 1 1 5BD61EFC
+P 9150 5650
+F 0 "#PWR0119" H 9150 5500 50  0001 C CNN
+F 1 "+24V" H 9165 5823 50  0000 C CNN
+F 2 "" H 9150 5650 50  0001 C CNN
+F 3 "" H 9150 5650 50  0001 C CNN
+	1    9150 5650
+	-1   0    0    1
+$EndComp
+Wire Wire Line
+	9150 5650 9150 5450
+$Comp
+L power:+5V #PWR0120
+U 1 1 5BD63789
+P 5450 3650
+F 0 "#PWR0120" H 5450 3500 50  0001 C CNN
+F 1 "+5V" H 5465 3823 50  0000 C CNN
+F 2 "" H 5450 3650 50  0001 C CNN
+F 3 "" H 5450 3650 50  0001 C CNN
+	1    5450 3650
+	1    0    0    -1
+$EndComp
 $EndSCHEMATC

Commit message: Add remaining connections.
Parts:
- added C?: C, symbol Device:C
- U2: footprint (none) -> Package_SO:TSSOP-14_4.4x5mm_P0.65mm
Connections:
- net labels added: IO18, IO19, IO23, IO5
- wire segments 74 -> 115
- no-connect marks 16 -> 27
Changed lines of the file:
@@
 F 0 "U2" H 3350 5815 50  0000 C CNN
 F 1 "74HCT08" H 3350 5724 50  0000 C CNN
-F 2 "" H 3350 5450 50  0001 C CNN
+F 2 "Package_SO:TSSOP-14_4.4x5mm_P0.65mm" H 3350 5450 50  0001 C CNN
 F 3 "" H 3350 5450 50  0001 C CNN
 	2    3350 5450
@@
 F 0 "U2" H 3350 6615 50  0000 C CNN
 F 1 "74HCT08" H 3350 6524 50  0000 C CNN
-F 2 "" H 3350 6250 50  0001 C CNN
+F 2 "Package_SO:TSSOP-14_4.4x5mm_P0.65mm" H 3350 6250 50  0001 C CNN
 F 3 "" H 3350 6250 50  0001 C CNN
 	3    3350 6250
@@
 Wire Wire Line
 	5450 3650 5450 3750
-Text GLabel 4550 3200 2    50   Input ~ 0
+Text GLabel 4250 3100 2    50   Input ~ 0
 SDA
-Text GLabel 4550 3300 2    50   Input ~ 0
+Text GLabel 4250 3200 2    50   Input ~ 0
 SCL
-Text GLabel 4500 3550 2    50   Input ~ 0
+Text GLabel 2900 4500 3    50   Input ~ 0
 MOSI
-Text GLabel 4500 3650 2    50   Input ~ 0
+Text GLabel 2800 4500 3    50   Input ~ 0
 MISO
-Text GLabel 4500 3750 2    50   Input ~ 0
+Text GLabel 3000 4500 3    50   Input ~ 0
 SCK
-Text GLabel 4500 3850 2    50   Input ~ 0
+Text GLabel 4250 2700 2    50   Input ~ 0
 CE
-Text GLabel 4500 3950 2    50   Input ~ 0
+Text GLabel 4250 2800 2    50   Input ~ 0
 CS
-Text GLabel 1150 2150 0    50   Input ~ 0
+Text GLabel 4250 4000 2    50   Input ~ 0
 EN
-Text GLabel 1150 2800 0    50   Input ~ 0
+Text GLabel 4250 3400 2    50   Input ~ 0
 Brake
 $Comp
@@
 F 0 "U2" H 3350 7515 50  0000 C CNN
 F 1 "74HCT08" H 3350 7424 50  0000 C CNN
-F 2 "" H 3350 7150 50  0001 C CNN
+F 2 "Package_SO:TSSOP-14_4.4x5mm_P0.65mm" H 3350 7150 50  0001 C CNN
 F 3 "" H 3350 7150 50  0001 C CNN
 	4    3350 7150
@@
 	1    0    0    -1
 $EndComp
+$Comp
+L power:GND #PWR?
+U 1 1 5BD50D91
+P 2050 4300
+F 0 "#PWR?" H 2050 4050 50  0001 C CNN
+F 1 "GND" H 2055 4127 50  0000 C CNN
+F 2 "" H 2050 4300 50  0001 C CNN
+F 3 "" H 2050 4300 50  0001 C CNN
+	1    2050 4300
+	1    0    0    -1
+$EndComp
+Wire Wire Line
+	2050 4300 2050 4100
+Wire Wire Line
+	2050 3900 2200 3900
+Wire Wire Line
+	2200 4000 2050 4000
+Connection ~ 2050 4000
+Wire Wire Line
+	2050 4000 2050 3900
+Wire Wire Line
+	2200 4100 2050 4100
+Connection ~ 2050 4100
+Wire Wire Line
+	2050 4100 2050 4000
+$Comp
+L Device:C C?
+U 1 1 5BD55B4E
+P 1850 3200
+F 0 "C?" H 1965 3246 50  0000 L CNN
+F 1 "C" H 1965 3155 50  0000 L CNN
+F 2 "" H 1888 3050 50  0001 C CNN
+F 3 "~" H 1850 3200 50  0001 C CNN
+	1    1850 3200
+	1    0    0    -1
+$EndComp
+$Comp
+L power:+5V #PWR?
+U 1 1 5BD55BFD
+P 1850 2850
+F 0 "#PWR?" H 1850 2700 50  0001 C CNN
+F 1 "+5V" H 1865 3023 50  0000 C CNN
+F 2 "" H 1850 2850 50  0001 C CNN
+F 3 "" H 1850 2850 50  0001 C CNN
+	1    1850 2850
+	1    0    0    -1
+$EndComp
+Wire Wire Line
+	1850 2850 1850 2950
+Wire Wire Line
+	2200 2950 1850 2950
+Connection ~ 1850 2950
+Wire Wire Line
+	1850 2950 1850 3050
+$Comp
+L power:GND #PWR?
+U 1 1 5BD59785
+P 1850 3450
+F 0 "#PWR?" H 1850 3200 50  0001 C CNN
+F 1 "GND" H 1855 3277 50  0000 C CNN
+F 2 "" H 1850 3450 50  0001 C CNN
+F 3 "" H 1850 3450 50  0001 C CNN
+	1    1850 3450
+	1    0    0    -1
+$EndComp
+Wire Wire Line
+	1850 3450 1850 3350
+$Comp
+L power:+3.3V #PWR?
+U 1 1 5BD5B963
+P 2100 2650
+F 0 "#PWR?" H 2100 2500 50  0001 C CNN
+F 1 "+3.3V" H 2115 2823 50  0000 C CNN
+F 2 "" H 2100 2650 50  0001 C CNN
+F 3 "" H 2100 2650 50  0001 C CNN
+	1    2100 2650
+	1    0    0    -1
+$EndComp
+Wire Wire Line
+	2100 2650 2100 2850
+Wire Wire Line
+	2100 2850 2200 2850
+Text GLabel 4700 1400 0    50   Input ~ 0
+IO5
+Text GLabel 3100 4550 3    50   Input ~ 0
+IO5
+Wire Wire Line
+	3100 4550 3100 4400
+Wire Wire Line
+	4800 1400 4700 1400
+Text GLabel 4700 1500 0    50   Input ~ 0
+IO18
+Text GLabel 4700 1600 0    50   Input ~ 0
+IO19
+Text GLabel 4700 1700 0    50   Input ~ 0
+IO23
+Wire Wire Line
+	4700 1700 4800 1700
+Wire Wire Line
+	4800 1600 4700 1600
+Wire Wire Line
+	4700 1500 4800 1500
+Text GLabel 4250 2900 2    50   Input ~ 0
+IO18
+Text GLabel 4250 3000 2    50   Input ~ 0
+IO19
+Text GLabel 4250 3300 2    50   Input ~ 0
+IO23
+Wire Wire Line
+	4250 3300 4150 3300
+Wire Wire Line
+	4250 3000 4150 3000
+Wire Wire Line
+	4250 2900 4150 2900
+Wire Wire Line
+	4800 1800 4700 1800
+Wire Wire Line
+	4700 1800 4700 1900
+Connection ~ 4700 2300
+Wire Wire Line
+	4800 1900 4700 1900
+Connection ~ 4700 1900
+Wire Wire Line
+	4700 1900 4700 2000
+Wire Wire Line
+	4800 2000 4700 2000
+Connection ~ 4700 2000
+Wire Wire Line
+	4700 2000 4700 2100
+Wire Wire Line
+	4800 2100 4700 2100
+Connection ~ 4700 2100
+Wire Wire Line
+	4700 2100 4700 2300
+NoConn ~ 5800 1800
+NoConn ~ 5800 1900
+NoConn ~ 5800 2000
+NoConn ~ 5800 2100
+Wire Wire Line
+	4250 3100 4150 3100
+Wire Wire Line
+	4150 3200 4250 3200
+Wire Wire Line
+	4250 2800 4150 2800
+Wire Wire Line
+	4150 2700 4250 2700
+Wire Wire Line
+	2800 4400 2800 4500
+Wire Wire Line
+	2900 4400 2900 4500
+Wire Wire Line
+	3000 4400 3000 4500
+Wire Wire Line
+	4250 4000 4150 4000
+Wire Wire Line
+	4150 3400 4250 3400
+NoConn ~ 2200 3550
+NoConn ~ 2200 3650
+NoConn ~ 4150 3500
+NoConn ~ 4150 3600
+NoConn ~ 4150 3700
+NoConn ~ 4150 3800
+NoConn ~ 4150 3900
+$Comp
+L power:+5V #PWR?
+U 1 1 5BDC7A11
+P 2650 6050
+F 0 "#PWR?" H 2650 5900 50  0001 C CNN
+F 1 "+5V" H 2665 6223 50  0000 C CNN
+F 2 "" H 2650 6050 50  0001 C CNN
+F 3 "" H 2650 6050 50  0001 C CNN
+	1    2650 6050
+	1    0    0    -1
+$EndComp
+Wire Wire Line
+	2650 6050 2650 6150
+Wire Wire Line
+	2650 6350 2800 6350
+Wire Wire Line
+	2800 6150 2650 6150
+Connection ~ 2650 6150
+Wire Wire Line
+	2650 6150 2650 6350
 $EndSCHEMATC

Commit message: Work on PCB.
Parts:
- added C10: 100n, Capacitor_SMD:C_0603_1608Metric, symbol Device:C
- added U9: PCA9515, Package_SO:TSSOP-8_3x3mm_P0.65mm, symbol pca9515:PCA9515
- C9: renamed from C?; value C -> 10u; footprint (none) -> Capacitor_SMD:C_0805_2012Metric
Connections:
- net labels added: SCL0, SCL1, SDA0, SDA1
- net labels removed: SCL, SDA
- wire segments 115 -> 125
- no-connect marks 27 -> 28
Changed lines of the file:
@@
 	5950 1000 5950 1050
 $Sheet
-S 8550 1500 500  150
+S 900  900  500  150
 U 5BC5FAEF
 F0 "Motor driver" 50
@@
 	7850 3250 7850 3350
 Text GLabel 5250 3950 0    50   Input ~ 0
-SDA
+SDA1
 Text GLabel 5250 4050 0    50   Input ~ 0
-SCL
+SCL1
 Wire Wire Line
 	5250 4050 5450 4050
@@
 	5450 3650 5450 3750
 Text GLabel 4250 3100 2    50   Input ~ 0
-SDA
+SDA0
 Text GLabel 4250 3200 2    50   Input ~ 0
-SCL
+SCL0
 Text GLabel 2900 4500 3    50   Input ~ 0
 MOSI
@@
 SCK
 Text GLabel 4250 2700 2    50   Input ~ 0
+CS
+Text GLabel 4250 2800 2    50   Input ~ 0
 CE
-Text GLabel 4250 2800 2    50   Input ~ 0
-CS
 Text GLabel 4250 4000 2    50   Input ~ 0
 EN
@@
 $EndComp
 $Comp
-L power:GND #PWR?
+L power:GND #PWR0121
 U 1 1 5BD50D91
 P 2050 4300
-F 0 "#PWR?" H 2050 4050 50  0001 C CNN
+F 0 "#PWR0121" H 2050 4050 50  0001 C CNN
 F 1 "GND" H 2055 4127 50  0000 C CNN
 F 2 "" H 2050 4300 50  0001 C CNN
@@
 	2050 4100 2050 4000
 $Comp
-L Device:C C?
+L Device:C C9
 U 1 1 5BD55B4E
 P 1850 3200
-F 0 "C?" H 1965 3246 50  0000 L CNN
-F 1 "C" H 1965 3155 50  0000 L CNN
-F 2 "" H 1888 3050 50  0001 C CNN
+F 0 "C9" H 1965 3246 50  0000 L CNN
+F 1 "10u" H 1965 3155 50  0000 L CNN
+F 2 "Capacitor_SMD:C_0805_2012Metric" H 1888 3050 50  0001 C CNN
 F 3 "~" H 1850 3200 50  0001 C CNN
 	1    1850 3200
@@
 $EndComp
 $Comp
-L power:+5V #PWR?
+L power:+5V #PWR0122
 U 1 1 5BD55BFD
 P 1850 2850
-F 0 "#PWR?" H 1850 2700 50  0001 C CNN
+F 0 "#PWR0122" H 1850 2700 50  0001 C CNN
 F 1 "+5V" H 1865 3023 50  0000 C CNN
 F 2 "" H 1850 2850 50  0001 C CNN
@@
 	1850 2950 1850 3050
 $Comp
-L power:GND #PWR?
+L power:GND #PWR0123
 U 1 1 5BD59785
 P 1850 3450
-F 0 "#PWR?" H 1850 3200 50  0001 C CNN
+F 0 "#PWR0123" H 1850 3200 50  0001 C CNN
 F 1 "GND" H 1855 3277 50  0000 C CNN
 F 2 "" H 1850 3450 50  0001 C CNN
@@
 	1850 3450 1850 3350
 $Comp
-L power:+3.3V #PWR?
+L power:+3.3V #PWR0124
 U 1 1 5BD5B963
 P 2100 2650
-F 0 "#PWR?" H 2100 2500 50  0001 C CNN
+F 0 "#PWR0124" H 2100 2500 50  0001 C CNN
 F 1 "+3.3V" H 2115 2823 50  0000 C CNN
 F 2 "" H 2100 2650 50  0001 C CNN
@@
 NoConn ~ 4150 3900
 $Comp
-L power:+5V #PWR?
+L power:+5V #PWR0125
 U 1 1 5BDC7A11
 P 2650 6050
-F 0 "#PWR?" H 2650 5900 50  0001 C CNN
+F 0 "#PWR0125" H 2650 5900 50  0001 C CNN
 F 1 "+5V" H 2665 6223 50  0000 C CNN
 F 2 "" H 2650 6050 50  0001 C CNN
@@
 Wire Wire Line
 	2650 6150 2650 6350
+$Comp
+L pca9515:PCA9515 U9
+U 1 1 5BD7A741
+P 8650 1700
+F 0 "U9" H 8250 2100 50  0000 C CNN
+F 1 "PCA9515" H 8150 2000 50  0000 C CNN
+F 2 "Package_SO:TSSOP-8_3x3mm_P0.65mm" H 8250 2050 50  0001 C CNN
+F 3 "http://www.ti.com/lit/ds/symlink/pca9306.pdf" H 8350 2150 50  0001 C CNN
+	1    8650 1700
+	1    0    0    -1
+$EndComp
+Text GLabel 7950 1700 0    50   Input ~ 0
+SCL0
+Text GLabel 7950 1800 0    50   Input ~ 0
+SDA0
+Text GLabel 9300 1700 2    50   Input ~ 0
+SCL1
+Text GLabel 9300 1800 2    50   Input ~ 0
+SDA1
+Wire Wire Line
+	9300 1800 9050 1800
+Wire Wire Line
+	9050 1700 9300 1700
+Wire Wire Line
+	8250 1700 7950 1700
+Wire Wire Line
+	7950 1800 8250 1800
+$Comp
+L power:GND #PWR09
+U 1 1 5BD8B088
+P 8650 2300
+F 0 "#PWR09" H 8650 2050 50  0001 C CNN
+F 1 "GND" H 8655 2127 50  0000 C CNN
+F 2 "" H 8650 2300 50  0001 C CNN
+F 3 "" H 8650 2300 50  0001 C CNN
+	1    8650 2300
+	1    0    0    -1
+$EndComp
+Wire Wire Line
+	8650 2300 8650 2200
+$Comp
+L Device:C C10
+U 1 1 5BD8F4AC
+P 9000 1100
+F 0 "C10" V 8748 1100 50  0000 C CNN
+F 1 "100n" V 8839 1100 50  0000 C CNN
+F 2 "Capacitor_SMD:C_0603_1608Metric" H 9038 950 50  0001 C CNN
+F 3 "~" H 9000 1100 50  0001 C CNN
+	1    9000 1100
+	0    1    1    0
+$EndComp
+$Comp
+L power:+3.3V #PWR01
+U 1 1 5BD8F5F9
+P 8650 1050
+F 0 "#PWR01" H 8650 900 50  0001 C CNN
+F 1 "+3.3V" H 8665 1223 50  0000 C CNN
+F 2 "" H 8650 1050 50  0001 C CNN
+F 3 "" H 8650 1050 50  0001 C CNN
+	1    8650 1050
+	1    0    0    -1
+$EndComp
+Wire Wire Line
+	8650 1050 8650 1100
+Wire Wire Line
+	8850 1100 8650 1100
+Connection ~ 8650 1100
+Wire Wire Line
+	8650 1100 8650 1200
+$Comp
+L power:GND #PWR010
+U 1 1 5BD98012
+P 9250 1200
+F 0 "#PWR010" H 9250 950 50  0001 C CNN
+F 1 "GND" H 9255 1027 50  0000 C CNN
+F 2 "" H 9250 1200 50  0001 C CNN
+F 3 "" H 9250 1200 50  0001 C CNN
+	1    9250 1200
+	1    0    0    -1
+$EndComp
+Wire Wire Line
+	9250 1200 9250 1100
+Wire Wire Line
+	9250 1100 9150 1100
+NoConn ~ 9050 1500
 $EndSCHEMATC

Commit message: Do more routing.
Connections:
- net labels added: IS_A_L_P, IS_A_R_P, IS_B_L_P, IS_B_R_P
- wire segments 125 -> 129
- no-connect marks 28 -> 24
Changed lines of the file:
@@
 $EndSheet
 Text GLabel 6150 1400 2    50   Input ~ 0
+PWM_A_R
+Text GLabel 6150 1500 2    50   Input ~ 0
 PWM_A_L
-Text GLabel 6150 1500 2    50   Input ~ 0
-PWM_A_R
 Text GLabel 6150 1600 2    50   Input ~ 0
 PWM_B_L
@@
 NoConn ~ 2200 3550
 NoConn ~ 2200 3650
-NoConn ~ 4150 3500
 NoConn ~ 4150 3600
-NoConn ~ 4150 3700
-NoConn ~ 4150 3800
-NoConn ~ 4150 3900
 $Comp
 L power:+5V #PWR0125
@@
 	9250 1100 9150 1100
 NoConn ~ 9050 1500
+Text GLabel 4250 3800 2    50   Input ~ 0
+IS_B_R_P
+Text GLabel 4250 3900 2    50   Input ~ 0
+IS_B_L_P
+Wire Wire Line
+	4150 3800 4250 3800
+Wire Wire Line
+	4250 3900 4150 3900
+Text GLabel 4250 3500 2    50   Input ~ 0
+IS_A_L_P
+Text GLabel 4250 3700 2    50   Input ~ 0
+IS_A_R_P
+Wire Wire Line
+	4150 3500 4250 3500
+Wire Wire Line
+	4250 3700 4150 3700
 $EndSCHEMATC

Commit message: Finalize layout.
Changed lines of the file:
@@
 PWM_A_L
 Text GLabel 6150 1600 2    50   Input ~ 0
+PWM_B_R
+Text GLabel 6150 1700 2    50   Input ~ 0
 PWM_B_L
-Text GLabel 6150 1700 2    50   Input ~ 0
-PWM_B_R
 Wire Wire Line
 	5800 1700 6150 1700
