File: pcb/chairbot/motor.kicad_sch (KiCad schematic)
At the start: 13 parts, among them J3 Conn_01x02, Q1 ZXMN4A06G, U6 Motor_driver, U7 Motor_driver

Commit message: Fix errors.
Connections:
- net EN is gone; now on net EN5: R1.2, R2.2
Changed lines of the file:
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@@
+	)
+	(junction
+		(at 135.89 46.99)
+		(diameter 0)
+		(color 0 0 0 0)
 	)
 	(junction
@@
 	(wire
 		(pts
-			(xy 120.65 54.61) (xy 135.89 54.61)
-		)
-		(stroke
-			(width 0)
-			(type default)
-		)
-	)
-	(wire
-		(pts
 			(xy 170.18 137.16) (xy 171.45 137.16)
 		)
@@
 	(wire
 		(pts
+			(xy 135.89 46.99) (xy 135.89 137.16)
+		)
+		(stroke
+			(width 0)
+			(type default)
+		)
+	)
+	(wire
+		(pts
 			(xy 189.23 30.48) (xy 203.2 30.48)
 		)
@@
 	(wire
 		(pts
-			(xy 135.89 54.61) (xy 135.89 137.16)
-		)
-		(stroke
-			(width 0)
-			(type default)
-		)
-	)
-	(wire
-		(pts
 			(xy 120.65 74.93) (xy 166.37 74.93)
 		)
@@
 	(wire
 		(pts
+			(xy 135.89 46.99) (xy 171.45 46.99)
+		)
+		(stroke
+			(width 0)
+			(type default)
+		)
+	)
+	(wire
+		(pts
 			(xy 179.07 127) (xy 182.88 127)
 		)
@@
 	(wire
 		(pts
-			(xy 120.65 46.99) (xy 171.45 46.99)
+			(xy 120.65 46.99) (xy 135.89 46.99)
 		)
 		(stroke
@@
 			(hide yes)
 			(show_name no)
-			(do_not_autoplace no)
-			(effects
-				(font
-					(size 1.27 1.27)
-				)
-			)
-		)
-	)
-	(global_label "EN"
-		(shape input)
-		(at 120.65 54.61 180)
-		(effects
-			(font
-				(size 1.27 1.27)
-			)
-			(justify right)
-		)
-		(property "Intersheetrefs" "${INTERSHEET_REFS}"
-			(at 120.65 54.61 0)
-			(hide yes)
-			(show_name no)
