File: pcb/chairbot/chairbot.kicad_pcb (KiCad board)
At the start: 2 copper layers, 66.9 x 100 mm, 34 parts, among them J1 Conn_01x02, J2 Conn_01x05, J3 Conn_01x02, J6 Micro_SD_Card_Det1, Q1 ZXMN4A06G, U1 ESP32mini, U2 PCM5102A module, U3 74HCT244, U4 buck-converter, U6 Motor_driver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

Commit message: Final touches.
Other:
- board text added: "24V"
- board text added: "Brake"
- board text added: "GND"
- board text added: "I2C"
- board text added: "USB"
Changed lines of the file:
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@@
 		(sheetname "/")
 		(sheetfile "chairbot.kicad_sch")
-		(units
-			(unit
-				(name "A")
-				(pins "16" "35" "2" "4" "5" "21" "23" "1" "22" "33" "34" "36" "32" "14"
-					"3" "15" "30" "39" "38" "18" "19" "40" "37" "20" "13" "17" "31" "29"
-					"8" "10" "27" "25" "12" "26" "6" "24" "28" "9" "11" "7"
-				)
-			)
-		)
 		(attr through_hole)
 		(duplicate_pad_numbers_are_jumpers no)
@@
 		(fp_line
 			(start -1.8 34.81)
-			(end 29.75 34.81)
+			(end 20 34.81)
 			(stroke
 				(width 0.05)
@@
 		)
 		(embedded_fonts no)
-		(model "${KISYS3DMOD}/Connector_PinHeader_2.54mm.3dshapes/PinHeader_2x10_P2.54mm_Vertical.step"
+		(model "${KISYS3DMOD}/Connector_PinSocket_2.54mm.3dshapes/PinSocket_2x10_P2.54mm_Vertical.step"
 			(offset
-				(xyz 0 0 0)
+				(xyz 27.5 0 0)
 			)
 			(scale
@@
 			)
 			(rotate
-				(xyz 0 0 0)
+				(xyz -0 -0 -0)
+			)
+		)
+		(model "${KISYS3DMOD}/Connector_PinSocket_2.54mm.3dshapes/PinSocket_2x10_P2.54mm_Vertical.step"
+			(offset
+				(xyz 3 0 0)
+			)
+			(scale
+				(xyz 1 1 1)
+			)
+			(rotate
+				(xyz -0 -0 -0)
 			)
 		)
@@
 		)
 		(embedded_fonts no)
-		(model "${KISYS3DMOD}/Connector_JST.3dshapes/JST_XH_B05B-XH-A_1x05_P2.50mm_Vertical.step"
+		(model "${KISYS3DMOD}/Connector_JST.3dshapes/JST_XH_B02B-XH-A_1x05_P2.50mm_Vertical.step"
+			(offset
+				(xyz 0 0 0)
+			)
+			(scale
+				(xyz 1 1 1)
+			)
+			(rotate
+				(xyz 0 0 0)
+			)
+		)
+		(model "${KICAD10_3DMODEL_DIR}/Connector_JST.3dshapes/JST_XH_B5B-XH-A_1x05_P2.50mm_Vertical.step"
 			(offset
 				(xyz 0 0 0)
@@
 		)
 		(embedded_fonts no)
+		(model "${KICAD10_3DMODEL_DIR}/Connector_Card.3dshapes/microSD_HC_Hirose_DM3D-SF.step"
+			(offset
+				(xyz -0.5 0 0)
+			)
+			(scale
+				(xyz 1 1 1)
+			)
+			(rotate
+				(xyz -0 -0 -0)
+			)
+		)
 	)
 	(footprint "MountingHole:MountingHole_3.2mm_M3"
@@
 			(at 0.7 2.5 0)
 			(layer "F.SilkS")
+			(hide yes)
 			(effects
 				(font
@@
 		)
 		(embedded_fonts no)
+		(model "${KICAD10_3DMODEL_DIR}/Connector_PinSocket_2.54mm.3dshapes/PinSocket_1x09_P2.54mm_Vertical.step"
+			(offset
+				(xyz -7.6 -6.5 0)
+			)
+			(scale
+				(xyz 1 1 1)
+			)
+			(rotate
+				(xyz -0 -0 -90)
+			)
+		)
+		(model "${KICAD10_3DMODEL_DIR}/Connector_PinSocket_2.54mm.3dshapes/PinSocket_1x06_P2.54mm_Vertical.step"
+			(offset
+				(xyz -14 6.5 0)
+			)
+			(scale
+				(xyz 1 1 1)
+			)
+			(rotate
+				(xyz -0 -0 -0)
+			)
+		)
 	)
 	(gr_line
@@
 		(layer "Edge.Cuts")
 	)
+	(gr_text "USB"
+		(at 74.422 123.698 0)
+		(layer "F.SilkS")
+		(effects
+			(font
+				(size 1 1)
+				(thickness 0.15)
+			)
+			(justify left bottom)
+		)
+	)
+	(gr_text "24V"
+		(at 81.026 174.752 0)
+		(layer "F.SilkS")
+		(effects
+			(font
+				(size 1 1)
+				(thickness 0.15)
+			)
+			(justify left bottom)
+		)
+	)
+	(gr_text "GND"
+		(at 86.106 179.324 0)
+		(layer "F.SilkS")
+		(effects
+			(font
+				(size 1 1)
+				(thickness 0.15)
+			)
+			(justify left bottom)
+		)
+	)
+	(gr_text "I2C"
+		(at 96.012 91.44 0)
+		(layer "F.SilkS")
+		(effects
+			(font
+				(size 1 1)
+				(thickness 0.15)
+			)
+			(justify left bottom)
+		)
+	)
+	(gr_text "Brake"
+		(at 45.974 178.308 90)
+		(layer "F.SilkS")
+		(effects
+			(font
+				(size 1 1)
+				(thickness 0.15)
+			)
+			(justify left bottom)
+		)
+	)
 	(gr_text "https://github.com/bullestock/chairbot/"

Commit message: Order.
Other:
- rule pad_to_mask_clearance: -0.2 -> 0
Changed lines of the file:
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@@
 	)
 	(paper "A4")
+	(title_block
+		(comment 4 "AISLER Project ID: ZAUALNVT")
+	)
 	(layers
 		(0 "F.Cu" signal)
@@
 	)
 	(setup
-		(pad_to_mask_clearance -0.2)
-		(solder_mask_min_width 0.25)
+		(pad_to_mask_clearance 0)
 		(allow_soldermask_bridges_in_footprints no)
 		(tenting
@@
 		(filling no)
 		(pcbplotparams
-			(layerselection 0x00000000_00000000_0003d1fc_ffffffff)
+			(layerselection 0x00000000_00000000_5555555d_ffffffff)
 			(plot_on_all_layers_selection 0x00000000_00000000_00000000_00000000)
 			(disableapertmacros no)
 			(usegerberextensions no)
-			(usegerberattributes no)
+			(usegerberattributes yes)
 			(usegerberadvancedattributes no)
 			(creategerberjobfile no)
