File: pcb/peripherals/peripherals.sch (KiCad schematic (older format))
At the start: 25 parts

Commit message: Start PCB layout.
Parts:
- added C2: 100n, Capacitor_THT:C_Disc_D7.5mm_W5.0mm_P5.00mm, symbol Device:C
- added C3: 100u, Capacitor_THT:CP_Radial_D8.0mm_P5.00mm, symbol Device:CP
- C1: renamed from C?; value CP -> 100u; footprint (none) -> Capacitor_THT:C_Radial_D12.5mm_H20.0mm_P5.00mm
- D1, D2: renamed from D?; footprint (none) -> Diode_THT:D_A-405_P10.16mm_Horizontal
- J1, J2: renamed from J?; footprint (none) -> Connector_JST:JST_XH_B05B-XH-A_1x05_P2.50mm_Vertical
- J10, J11, J9: renamed from J?; footprint (none) -> Connector_JST:JST_XH_B02B-XH-A_1x02_P2.50mm_Vertical
- J3, J4: renamed from J?; footprint (none) -> Connector_PinHeader_2.54mm:PinHeader_1x04_P2.54mm_Vertical
- J5, J6, J7, J8: renamed from J?; footprint (none) -> Connector_JST:JST_XH_B04B-XH-A_1x04_P2.50mm_Vertical
- Q1, Q2: renamed from Q?; footprint (none) -> Package_TO_SOT_THT:TO-220-3_Vertical
- R1, R2, R3, R4, R5, R6: renamed from R?; footprint (none) -> Resistor_THT:R_Axial_DIN0411_L9.9mm_D3.6mm_P25.40mm_Horizontal
- U1: renamed from U?; footprint (none) -> Peripherals:DFPlayer
- U2: renamed from U?; footprint mylib:buck-converter -> Peripherals:buck-converter
- gave numbers to parts that had none: 1
Connections:
- net +5V: now also C2.1
- net +5VP: now also C3.1
- net GND: now also C2.2, C3.2
- net at A1.19 (A0): now also U1.16 (BUSY)
- net at U1.4 (DAC_R): now also J3.2 (Pin_2)
- net at U1.5 (DAC_L): now also J4.2 (Pin_2)
- net at U1.6 (SPK_1): no longer J3.2 (Pin_2)
- net at U1.8 (SPK_2): no longer J4.2 (Pin_2)
- no-connect marks 7 -> 20

Commit message: Route more tracks.
Parts:
- D1, D2: footprint Diode_THT:D_A-405_P10.16mm_Horizontal -> Diode_THT:D_A-405_P5.08mm_Vertical_KathodeUp
Changed lines of the file:
@@
 F 0 "D1" H 8450 3016 50  0000 C CNN
 F 1 "1N4001" H 8450 2925 50  0000 C CNN
-F 2 "Diode_THT:D_A-405_P10.16mm_Horizontal" H 8450 2800 50  0001 C CNN
+F 2 "Diode_THT:D_A-405_P5.08mm_Vertical_KathodeUp" H 8450 2800 50  0001 C CNN
 F 3 "~" H 8450 2800 50  0001 C CNN
 	1    8450 2800
@@
 F 0 "D2" H 8450 4766 50  0000 C CNN
 F 1 "1N4001" H 8450 4675 50  0000 C CNN
-F 2 "Diode_THT:D_A-405_P10.16mm_Horizontal" H 8450 4550 50  0001 C CNN
+F 2 "Diode_THT:D_A-405_P5.08mm_Vertical_KathodeUp" H 8450 4550 50  0001 C CNN
 F 3 "~" H 8450 4550 50  0001 C CNN
 	1    8450 4550

Commit message: Complete routing.
Parts:
- removed J5, J6, J7, J8: JST XH, Connector_JST:JST_XH_B04B-XH-A_1x04_P2.50mm_Vertical, symbol Connector_Generic:Conn_01x04
- added H1, H2, H3, H4: MountingHole, MountingHole:MountingHole_3.2mm_M3, symbol Mechanical:MountingHole
- R1, R2, R3: footprint Resistor_THT:R_Axial_DIN0411_L9.9mm_D3.6mm_P25.40mm_Horizontal -> Resistor_THT:R_Axial_DIN0414_L11.9mm_D4.5mm_P5.08mm_Vertical
- R4: footprint Resistor_THT:R_Axial_DIN0411_L9.9mm_D3.6mm_P25.40mm_Horizontal -> Resistor_THT:R_Axial_DIN0414_L11.9mm_D4.5mm_P7.62mm_Vertical
Connections:
- net IO1: no longer names the net of A1.5 (D2)
- net IO2: no longer names the net of A1.6 (D3)
- net IO3: no longer names the net of A1.7 (D4)
- net IO4: no longer names the net of A1.8 (D5)
- net IO5: no longer names the net of A1.9 (D6)
- net IO6: no longer names the net of A1.10 (D7)
- net IO7: no longer names the net of A1.11 (D8)
- net IO8: no longer names the net of A1.12 (D9)
- no-connect marks 20 -> 28
Other:
- note added: "24V IN"
- note added: "PWM1 OUT"
- note added: "PWM2 OUT"
Changed lines of the file:
@@
 F 0 "R1" V 3550 3850 50  0000 C CNN
 F 1 "1k" V 3600 4050 50  0000 C CNN
-F 2 "Resistor_THT:R_Axial_DIN0411_L9.9mm_D3.6mm_P25.40mm_Horizontal" V 3530 4050 50  0001 C CNN
+F 2 "Resistor_THT:R_Axial_DIN0414_L11.9mm_D4.5mm_P5.08mm_Vertical" V 3530 4050 50  0001 C CNN
 F 3 "~" H 3600 4050 50  0001 C CNN
 	1    3600 4050
@@
 F 0 "R3" V 8000 3350 50  0000 L CNN
 F 1 "47k" V 8100 3400 50  0000 L CNN
-F 2 "Resistor_THT:R_Axial_DIN0411_L9.9mm_D3.6mm_P25.40mm_Horizontal" V 8030 3450 50  0001 C CNN
+F 2 "Resistor_THT:R_Axial_DIN0414_L11.9mm_D4.5mm_P5.08mm_Vertical" V 8030 3450 50  0001 C CNN
 F 3 "~" H 8100 3450 50  0001 C CNN
 	1    8100 3450
@@
 F 0 "R2" V 8000 3150 50  0000 C CNN
 F 1 "1k" V 8100 3200 50  0000 C CNN
-F 2 "Resistor_THT:R_Axial_DIN0411_L9.9mm_D3.6mm_P25.40mm_Horizontal" V 8030 3200 50  0001 C CNN
+F 2 "Resistor_THT:R_Axial_DIN0414_L11.9mm_D4.5mm_P5.08mm_Vertical" V 8030 3200 50  0001 C CNN
 F 3 "~" H 8100 3200 50  0001 C CNN
 	1    8100 3200
@@
 F 0 "R4" V 8000 4900 50  0000 C CNN
 F 1 "1k" V 8100 4950 50  0000 C CNN
-F 2 "Resistor_THT:R_Axial_DIN0411_L9.9mm_D3.6mm_P25.40mm_Horizontal" V 8030 4950 50  0001 C CNN
+F 2 "Resistor_THT:R_Axial_DIN0414_L11.9mm_D4.5mm_P7.62mm_Vertical" V 8030 4950 50  0001 C CNN
 F 3 "~" H 8100 4950 50  0001 C CNN
 	1    8100 4950
@@
 Wire Wire Line
 	5950 3950 6150 3950
-$Comp
-L Connector_Generic:Conn_01x04 J5
-U 1 1 5D2416E7
-P 3350 1050
-F 0 "J5" H 3268 1367 50  0000 C CNN
-F 1 "JST XH" H 3268 1276 50  0000 C CNN
-F 2 "Connector_JST:JST_XH_B04B-XH-A_1x04_P2.50mm_Vertical" H 3350 1050 50  0001 C CNN
-F 3 "~" H 3350 1050 50  0001 C CNN
-	1    3350 1050
-	-1   0    0    -1
-$EndComp
-$Comp
-L Connector_Generic:Conn_01x04 J6
-U 1 1 5D2427F5
-P 3350 1700
-F 0 "J6" H 3268 2017 50  0000 C CNN
-F 1 "JST XH" H 3268 1926 50  0000 C CNN
-F 2 "Connector_JST:JST_XH_B04B-XH-A_1x04_P2.50mm_Vertical" H 3350 1700 50  0001 C CNN
-F 3 "~" H 3350 1700 50  0001 C CNN
-	1    3350 1700
-	-1   0    0    -1
-$EndComp
-$Comp
-L power:+5V #PWR0118
-U 1 1 5D25421A
-P 3750 850
-F 0 "#PWR0118" H 3750 700 50  0001 C CNN
-F 1 "+5V" H 3765 1023 50  0000 C CNN
-F 2 "" H 3750 850 50  0001 C CNN
-F 3 "" H 3750 850 50  0001 C CNN
-	1    3750 850
-	1    0    0    -1
-$EndComp
-Wire Wire Line
-	3750 850  3750 950
-Wire Wire Line
-	3750 1600 3550 1600
-Wire Wire Line
-	3550 950  3750 950
-Connection ~ 3750 950
-Wire Wire Line
-	3750 950  3750 1600
-$Comp
-L power:GND #PWR0119
-U 1 1 5D25BE36
-P 3650 2050
-F 0 "#PWR0119" H 3650 1800 50  0001 C CNN
-F 1 "GND" H 3655 1877 50  0000 C CNN
-F 2 "" H 3650 2050 50  0001 C CNN
-F 3 "" H 3650 2050 50  0001 C CNN
-	1    3650 2050
-	1    0    0    -1
-$EndComp
-Wire Wire Line
-	3650 2050 3650 1900
-Wire Wire Line
-	3650 1250 3550 1250
-Wire Wire Line
-	3550 1900 3650 1900
-Connection ~ 3650 1900
-Wire Wire Line
-	3650 1900 3650 1250
-Text GLabel 3900 1050 2    50   Input ~ 0
-IO1
-Text GLabel 3900 1150 2    50   Input ~ 0
-IO2
-Text GLabel 3900 1700 2    50   Input ~ 0
-IO3
-Text GLabel 3900 1800 2    50   Input ~ 0
-IO4
-Wire Wire Line
-	3900 1800 3550 1800
-Wire Wire Line
-	3550 1700 3900 1700
-Wire Wire Line
-	3900 1150 3550 1150
-Wire Wire Line
-	3550 1050 3900 1050
-$Comp
-L Connector_Generic:Conn_01x04 J7
-U 1 1 5D27C554
-P 4550 1050
-F 0 "J7" H 4468 1367 50  0000 C CNN
-F 1 "JST XH" H 4468 1276 50  0000 C CNN
-F 2 "Connector_JST:JST_XH_B04B-XH-A_1x04_P2.50mm_Vertical" H 4550 1050 50  0001 C CNN
-F 3 "~" H 4550 1050 50  0001 C CNN
-	1    4550 1050
-	-1   0    0    -1
-$EndComp
-$Comp
-L Connector_Generic:Conn_01x04 J8
-U 1 1 5D27C55E
-P 4550 1700
-F 0 "J8" H 4468 2017 50  0000 C CNN
-F 1 "JST XH" H 4468 1926 50  0000 C CNN
-F 2 "Connector_JST:JST_XH_B04B-XH-A_1x04_P2.50mm_Vertical" H 4550 1700 50  0001 C CNN
-F 3 "~" H 4550 1700 50  0001 C CNN
-	1    4550 1700
-	-1   0    0    -1
-$EndComp
-$Comp
-L power:+5V #PWR0120
-U 1 1 5D27C568
-P 4950 850
-F 0 "#PWR0120" H 4950 700 50  0001 C CNN
-F 1 "+5V" H 4965 1023 50  0000 C CNN
-F 2 "" H 4950 850 50  0001 C CNN
-F 3 "" H 4950 850 50  0001 C CNN
-	1    4950 850
-	1    0    0    -1
-$EndComp
-Wire Wire Line
-	4950 850  4950 950
-Wire Wire Line
-	4950 1600 4750 1600
-Wire Wire Line
-	4750 950  4950 950
-Connection ~ 4950 950
-Wire Wire Line
-	4950 950  4950 1600
-$Comp
-L power:GND #PWR0121
-U 1 1 5D27C577
-P 4850 2050
-F 0 "#PWR0121" H 4850 1800 50  0001 C CNN
-F 1 "GND" H 4855 1877 50  0000 C CNN
-F 2 "" H 4850 2050 50  0001 C CNN
-F 3 "" H 4850 2050 50  0001 C CNN
-	1    4850 2050
-	1    0    0    -1
-$EndComp
-Wire Wire Line
-	4850 2050 4850 1900
-Wire Wire Line
-	4850 1250 4750 1250
-Wire Wire Line
-	4750 1900 4850 1900
-Connection ~ 4850 1900
-Wire Wire Line
-	4850 1900 4850 1250
-Text GLabel 5100 1050 2    50   Input ~ 0
-IO5
-Text GLabel 5100 1150 2    50   Input ~ 0
-IO6
-Text GLabel 5100 1700 2    50   Input ~ 0
-IO7
-Text GLabel 5100 1800 2    50   Input ~ 0
-IO8
-Wire Wire Line
-	5100 1800 4750 1800
-Wire Wire Line
-	4750 1700 5100 1700
-Wire Wire Line
-	5100 1150 4750 1150
-Wire Wire Line
-	4750 1050 5100 1050
-Text GLabel 4650 3150 0    50   Input ~ 0
-IO1
-Text GLabel 4650 3250 0    50   Input ~ 0
-IO2
-Text GLabel 4650 3350 0    50   Input ~ 0
-IO3
-Text GLabel 4650 3450 0    50   Input ~ 0
-IO4
-Text GLabel 4650 3550 0    50   Input ~ 0
-IO5
-Text GLabel 4650 3650 0    50   Input ~ 0
-IO6
-Text GLabel 4650 3750 0    50   Input ~ 0
-IO7
-Text GLabel 4650 3850 0    50   Input ~ 0
-IO8
-Wire Wire Line
-	4650 3850 4950 3850
-Wire Wire Line
-	4950 3750 4650 3750
-Wire Wire Line
-	4650 3650 4950 3650
-Wire Wire Line
-	4950 3550 4650 3550
-Wire Wire Line
-	4650 3450 4950 3450
-Wire Wire Line
-	4950 3350 4650 3350
-Wire Wire Line
-	4650 3250 4950 3250
-Wire Wire Line
-	4950 3150 4650 3150
 NoConn ~ 4950 2950
 NoConn ~ 4950 3050
@@
 	2400 4450 2700 4450
 Connection ~ 2700 4450
+NoConn ~ 4950 3150
+NoConn ~ 4950 3250
+NoConn ~ 4950 3350
+NoConn ~ 4950 3450
+NoConn ~ 4950 3550
+NoConn ~ 4950 3650
+NoConn ~ 4950 3750
+NoConn ~ 4950 3850
+$Comp
+L Mechanical:MountingHole H1
+U 1 1 5D1E466A
+P 2900 2650
+F 0 "H1" H 3000 2696 50  0000 L CNN
+F 1 "MountingHole" H 3000 2605 50  0000 L CNN
+F 2 "MountingHole:MountingHole_3.2mm_M3" H 2900 2650 50  0001 C CNN
+F 3 "~" H 2900 2650 50  0001 C CNN
+	1    2900 2650
+	1    0    0    -1
+$EndComp
+$Comp
+L Mechanical:MountingHole H2
+U 1 1 5D1E4A4A
+P 2900 2900
+F 0 "H2" H 3000 2946 50  0000 L CNN
+F 1 "MountingHole" H 3000 2855 50  0000 L CNN
+F 2 "MountingHole:MountingHole_3.2mm_M3" H 2900 2900 50  0001 C CNN
+F 3 "~" H 2900 2900 50  0001 C CNN
+	1    2900 2900
+	1    0    0    -1
+$EndComp
+$Comp
+L Mechanical:MountingHole H3
+U 1 1 5D1E4E06
+P 2900 3150
+F 0 "H3" H 3000 3196 50  0000 L CNN
+F 1 "MountingHole" H 3000 3105 50  0000 L CNN
+F 2 "MountingHole:MountingHole_3.2mm_M3" H 2900 3150 50  0001 C CNN
+F 3 "~" H 2900 3150 50  0001 C CNN
+	1    2900 3150
+	1    0    0    -1
+$EndComp
+$Comp
+L Mechanical:MountingHole H4
+U 1 1 5D1E53AF
+P 2900 3400
+F 0 "H4" H 3000 3446 50  0000 L CNN
+F 1 "MountingHole" H 3000 3355 50  0000 L CNN
+F 2 "MountingHole:MountingHole_3.2mm_M3" H 2900 3400 50  0001 C CNN
+F 3 "~" H 2900 3400 50  0001 C CNN
+	1    2900 3400
+	1    0    0    -1
+$EndComp
+Text Notes 9100 1400 0    50   ~ 0
+24V IN
+Text Notes 9050 2500 0    50   ~ 0
+PWM1 OUT
+Text Notes 9050 4250 0    50   ~ 0
+PWM2 OUT
 $EndSCHEMATC

Commit message: Update.
Connections:
- net PWM1: now also A1.6 (D3); no longer A1.15 (D12)
- net PWM2: now also A1.8 (D5); no longer A1.16 (D13)
Changed lines of the file:
@@
 Wire Wire Line
 	7800 4950 7950 4950
-Text GLabel 4650 4150 0    50   Input ~ 0
+Text GLabel 4650 3250 0    50   Input ~ 0
 PWM1
-Text GLabel 4650 4250 0    50   Input ~ 0
+Text GLabel 4650 3450 0    50   Input ~ 0
 PWM2
-Wire Wire Line
-	4650 4250 4950 4250
-Wire Wire Line
-	4950 4150 4650 4150
 Text GLabel 6150 3950 2    50   Input ~ 0
 SDA
@@
 Connection ~ 2700 4450
 NoConn ~ 4950 3150
-NoConn ~ 4950 3250
 NoConn ~ 4950 3350
-NoConn ~ 4950 3450
 NoConn ~ 4950 3550
 NoConn ~ 4950 3650
@@
 Text Notes 9050 4250 0    50   ~ 0
 PWM2 OUT
+Wire Wire Line
+	4650 3450 4950 3450
+Wire Wire Line
+	4950 3250 4650 3250
+NoConn ~ 4950 4150
+NoConn ~ 4950 4250
 $EndSCHEMATC

Commit message: SMD version.
Parts:
- removed D1, D2: 1N4001, Diode_THT:D_A-405_P5.08mm_Vertical_KathodeUp, symbol Device:D
- removed J10, J11: JST XH, Connector_JST:JST_XH_B02B-XH-A_1x02_P2.50mm_Vertical, symbol Connector_Generic:Conn_01x02
- removed J3, J4: Pin header, Connector_PinHeader_2.54mm:PinHeader_1x04_P2.54mm_Vertical, symbol Connector_Generic:Conn_01x04
- removed Q1, Q2: IRFZ44N, Package_TO_SOT_THT:TO-220-3_Vertical, symbol Device:Q_NMOS_GDS
- removed R2: 1k, Resistor_THT:R_Axial_DIN0414_L11.9mm_D4.5mm_P5.08mm_Vertical, symbol Device:R
- removed R3: 47k, Resistor_THT:R_Axial_DIN0414_L11.9mm_D4.5mm_P5.08mm_Vertical, symbol Device:R
- removed R4: 1k, Resistor_THT:R_Axial_DIN0414_L11.9mm_D4.5mm_P7.62mm_Vertical, symbol Device:R
- removed R5: 47k, Resistor_THT:R_Axial_DIN0411_L9.9mm_D3.6mm_P25.40mm_Horizontal, symbol Device:R
- removed U2: buck-converter, Peripherals:buck-converter, symbol buckconverter:buck-converter
- added C9: 1u, Capacitor_SMD:C_0805_2012Metric, symbol Device:C
- added J3: Conn_01x03, Connector_JST:JST_XH_B03B-XH-A_1x03_P2.50mm_Vertical, symbol Connector_Generic:Conn_01x03
- C1: footprint Capacitor_THT:C_Radial_D12.5mm_H20.0mm_P5.00mm -> Capacitor_SMD:CP_Elec_10x10
- C2: value 100n -> 1u; footprint Capacitor_THT:C_Disc_D7.5mm_W5.0mm_P5.00mm -> Capacitor_SMD:C_0603_1608Metric
- C3: footprint Capacitor_THT:CP_Radial_D8.0mm_P5.00mm -> Capacitor_SMD:CP_Elec_10x10
- R1: footprint Resistor_THT:R_Axial_DIN0414_L11.9mm_D4.5mm_P5.08mm_Vertical -> Resistor_SMD:R_0603_1608Metric
- R6: footprint Resistor_THT:R_Axial_DIN0411_L9.9mm_D3.6mm_P25.40mm_Horizontal -> Resistor_SMD:R_0603_1608Metric
Connections:
- net +5VP is gone; now on net +5V: C3.1
- net +5V: now also C9.2
- net GND: now also C9.1, J3.2 (Pin_2); no longer C1.2
- net GNDPWR: now also C1.2
- net PWM4: now reaches A1.12 (D9)
- net at A1.13 (D10): no longer U1.3 (TX)
- net at A1.14 (D11): no longer R1.1
- net DFTX: now reaches A1.21 (A2)
- net DFTX: now also U1.3 (TX)
- net DFRX: now reaches A1.22 (A3)
- net DFRX: now also R1.1
- net PWM3: now reaches A1.9 (D6)
- net at U1.4 (DAC_R): now also J3.3 (Pin_3)
- net at U1.5 (DAC_L): now also J3.1 (Pin_1)
- no-connect marks 28 -> 26
Other:
- note removed: "PWM1 OUT"
- note removed: "PWM2 OUT"
