File: pcb/peripherals/peripherals.kicad_pcb (KiCad board)
At the start: 2 copper layers, 76.5 x 61.8 mm, 42 parts, among them J1 JST XH, J10 Conn_01x04, J2 JST XH, J3 JST XH, J4 Conn_01x08, J5 JST XH, J6 JST XH, J7 JST XH, J8 JST XH, J9 Conn_01x08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

Commit message: Route UART to J10.
Parts:
- Q2, Q4, Q6, Q8: value IRFR5505TRPBF -> IRFR5505TRPBF
Connections:
- D1 pad 1: Net-(D1-Pad1) -> Net-(D1-K)
- D2 pad 1: Net-(D2-Pad1) -> Net-(D2-K)
- D3 pad 1: Net-(D3-Pad1) -> Net-(D3-K)
- D4 pad 1: Net-(D4-Pad1) -> Net-(D4-K)
- J10 pad 3: MPTX -> GRBLTX
- J10 pad 4: MPRX -> GRBLRX
- J5 pad 1: Net-(D1-Pad1) -> Net-(D1-K)
- J6 pad 1: Net-(D2-Pad1) -> Net-(D2-K)
- J7 pad 1: Net-(D3-Pad1) -> Net-(D3-K)
- J8 pad 1: Net-(D4-Pad1) -> Net-(D4-K)
- Q2 pad 2: Net-(D1-Pad1) -> +24V
- Q2 pad 3: +24V -> Net-(D1-K)
- Q4 pad 2: Net-(D2-Pad1) -> +24V
- Q4 pad 3: +24V -> Net-(D2-K)
- Q6 pad 2: Net-(D3-Pad1) -> +24V
- Q6 pad 3: +24V -> Net-(D3-K)
- Q8 pad 2: Net-(D4-Pad1) -> +24V
- Q8 pad 3: +24V -> Net-(D4-K)
- U1 pad 1: unconnected-(U1-Pad1) -> GRBLRX
- U1 pad 2: unconnected-(U1-Pad2) -> GRBLTX
- U1 pad 5: MPRX -> unconnected-(U1-D2-Pad5)
- U1 pad 7: MPTX -> unconnected-(U1-D4-Pad7)
Routing:
- net +24V: track 121.2 -> 201.3 mm
- net Net-(D1-Pad1): track 20.8 -> 0.00 mm
- net Net-(D4-Pad1): track 20.0 -> 0.00 mm
- net Net-(D3-Pad1): track 19.8 -> 0.00 mm
- net Net-(D2-Pad1): track 19.5 -> 0.00 mm
- net MPRX: track 6.90 -> 0.00 mm
- net MPTX: track 6.52 -> 0.00 mm
